File: connectors.kicad_sch (KiCad schematic)
At the start: 13 parts, among them J1 NC3MAV, J10 Output, J12 NC3MAAV-1, J2 AMASS_XT60-M_1x02_P7.20mm_Ver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, J3 AMASS_XT60-F_1x02_P7.20mm_Ver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, J4 TE_MATE-N-LOK_350211-1_1x04_P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, J5 TE_MATE-N-LOK_350211-1_1x04_P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, J6 NC3FAV, J7 Conn_01x03_Pin, J8 Conn_01x03_Pin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

Commit message: snap
Parts:
- added C22: 330uF 25V, Capacitor_SMD:CP_Elec_8x10.5, symbol Device:C
- added F1: 16V 1.5A, Fuse:Fuse_1206_3216Metric, symbol Device:Polyfuse
- added J11: ~, Connector_AMASS:AMASS_XT60PW-M_1x02_P7.20mm_Horizontal, symbol Connector:Conn_01x02_Pin
- added J13: ~, Connector_AMASS:AMASS_XT60PW-F_1x02_P7.20mm_Horizontal, symbol Connector:Conn_01x02_Socket
- added J14: Input, Connector_RJ:RJ45_RCH_RC01937, symbol Connector:8P8C_Shielded
- added J15: Output, Connector_RJ:RJ45_RCH_RC01937, symbol Connector:8P8C_Shielded
Connections:
- net D_{in}: now also J14.3, J14.6
- net D_{out}: now also J15.3, J15.6
- net GND: now also J10.SH, C22.2, J11.1 (Pin_1), J13.1 (Pin_1), J14.4, J14.5, J15.4, J15.5, J15.SH
- net Shield: now also J14.SH
- net VDD: now also C22.1, F1.2, J14.7, J14.8, J15.7, J15.8; no longer J2.2 (Pin_2), J3.2 (Pin_2)
- net at J10.1, J10.2: now also J15.1, J15.2
- net at J9.1, J9.2: now also J14.1, J14.2
- new net Vin: F1.1, J11.2 (Pin_2), J13.2 (Pin_2), J2.2 (Pin_2), J3.2 (Pin_2)
- no-connect marks 1 -> 0
Other:
- moved on the sheet: J2
