File: klopfer.kicad_sch (KiCad schematic)
At the start: 5 parts

Commit message: snap
Parts:
- renumbered C19 to C1, D19 to D1, N19 to N1, TP15 to TP1
Changed lines of the file:
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@@
 (kicad_sch
-	(version 20231120)
+	(version 20250114)
 	(generator "eeschema")
-	(generator_version "8.0")
+	(generator_version "9.0")
 	(paper "A4")
 	(junction
@@
 		(shape input)
 		(at 48.26 57.15 180)
-		(fields_autoplaced yes)
 		(effects
 			(font
@@
 		(shape output)
 		(at 73.66 57.15 0)
-		(fields_autoplaced yes)
 		(effects
 			(font
@@
 		(dnp no)
 		(fields_autoplaced yes)
-		(property "Reference" "#PWR094"
+		(property "Reference" "#PWR02"
 			(at 66.04 86.36 0)
 			(effects
@@
 		(dnp no)
 		(fields_autoplaced yes)
-		(property "Reference" "C19"
+		(property "Reference" "C1"
 			(at 88.9 54.6099 0)
 			(effects
@@
 		(dnp no)
 		(fields_autoplaced yes)
-		(property "Reference" "D19"
+		(property "Reference" "D1"
 			(at 80.01 50.8314 0)
 			(effects
@@
 		(dnp no)
 		(fields_autoplaced yes)
-		(property "Reference" "#PWR093"
+		(property "Reference" "#PWR01"
 			(at 66.04 34.29 0)
 			(effects
@@
 		(dnp no)
 		(fields_autoplaced yes)
-		(property "Reference" "TP15"
+		(property "Reference" "TP1"
 			(at 52.07 48.26 0)
 			(effects
@@
 		(dnp no)
 		(fields_autoplaced yes)
-		(property "Reference" "N19"
+		(property "Reference" "N1"
 			(at 113.03 44.7674 0)
 			(effects
